File: custom-pcb/custom-pcb.sch (KiCad schematic (older format))
At the start: 67 parts, among them J1 CONN_CTL, J2 CONN_UART, J3 CONN_DBRD_IN, J4 CONN_DBRD_OUT, SW1 RESET, SW10 RESET_D, SW11 BOOT_D, SW2 BOOT, SW3 SPR_POWER, SW4 SPR_FAN, SW5 SPR_NIGHT, SW6 SPR_TIMER, SW7 SPR_FILTER, SW8 SPR_LIGHT, SW9 SPR_LOCK, U1 AMS1117-3.3, U2 74HCT595PW,118, U3 74HCT595PW,118, U4 ESP32-WROOM-32

Commit message: Increase EN capacitor value
Parts:
- C5: value 0u1 -> 10u
Changed lines of the file:
@@
 Sheet 1 1
 Title "Levoit Purifier ESP32 PCB"
-Date "2021-04-13"
-Rev "v0.1"
+Date "2021-05-18"
+Rev "v0.2"
 Comp "Davide Depau"
 Comment1 ""
@@
 P 5050 1350
 F 0 "C5" H 5142 1396 50  0000 L CNN
-F 1 "0u1" H 5142 1305 50  0000 L CNN
+F 1 "10u" H 5142 1305 50  0000 L CNN
 F 2 "Capacitor_SMD:C_0402_1005Metric" H 5050 1350 50  0001 C CNN
 F 3 "~" H 5050 1350 50  0001 C CNN

Commit message: Add LED filter caps and touchpad series res
Parts:
- added C? (x13): 0u1, symbol Device:C_Small
- added R? (x7): 510R, symbol Device:R_Small
- D1, D10, D11, D12, D13, D2, D3, D4, D5, D6, D7, D8, D9: footprint LED_THT:LED_D5.0mm -> custom-pcb:LED_D5.0mm-centered
Connections:
- net GND: now also C?.1, C?.1, C?.1, C?.1, C?.1, C?.1, C?.1, C?.1, C?.1, C?.1, C?.1, C?.1, C?.1
- net LED_BLUE_2H: now also C?.2
- net LED_BLUE_4H: now also C?.2
- net LED_BLUE_6H: now also C?.2
- net LED_BLUE_8H: now also C?.2
- net LED_BLUE_V1: now also C?.2
- net LED_BLUE_V2: now also C?.2
- net LED_BLUE_V3: now also C?.2
- net LED_RED_FILTER: now also C?.2
- net LED_WHITE_FAN: now also C?.2
- net LED_WHITE_LOCK: now also C?.2
- net LED_WHITE_NIGHT: now also C?.2
- net LED_WHITE_POWER: now also C?.2
- net LED_WHITE_TIMER: now also C?.2
- net TOUCH_FAN: now also R?.2; no longer SW4.1 (IN)
- net TOUCH_FILTER: now also R?.2; no longer SW7.1 (IN)
- net TOUCH_LIGHT: now also R?.2; no longer SW8.1 (IN)
- net TOUCH_LOCK: now also R?.2; no longer SW9.1 (IN)
- net TOUCH_NIGHT: now also R?.2; no longer SW5.1 (IN)
- net TOUCH_POWER: now also R?.2; no longer SW3.1 (IN)
- net TOUCH_TIMER: now also R?.2; no longer SW6.1 (IN)
- new net: R?.1, SW3.1 (IN)
- new net: R?.1, SW5.1 (IN)
- new net: R?.1, SW8.1 (IN)
- new net: R?.1, SW4.1 (IN)
- new net: R?.1, SW6.1 (IN)
- new net: R?.1, SW9.1 (IN)
- new net: R?.1, SW7.1 (IN)
Other:
- moved on the sheet: C7, C8, D10, D11, D12, D13, D6, D8, D9, J1, J2, J3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

Commit message: Change blue LED footprints to SMD
Parts:
- C10, C11, C12, C13, C14, C15, C16, C17, C18, C19, C20, C21, C9: renamed from C?; footprint (none) -> Capacitor_SMD:C_0402_1005Metric
- D10, D12, D5, D6, D7, D8, D9: footprint custom-pcb:LED_D5.0mm-centered -> LED_SMD:LED_0603_1608Metric_Pad1.05x0.95mm_HandSolder
- R28, R29, R30, R31, R32, R33, R34: renamed from R?; footprint (none) -> Resistor_SMD:R_0402_1005Metric
Changed lines of the file:
@@
 F 0 "D6" V 4446 5580 50  0000 R CNN
 F 1 "LED_B_6H" V 4355 5580 50  0000 R CNN
-F 2 "custom-pcb:LED_D5.0mm-centered" V 4400 5650 50  0001 C CNN
+F 2 "LED_SMD:LED_0603_1608Metric_Pad1.05x0.95mm_HandSolder" V 4400 5650 50  0001 C CNN
 F 3 "~" V 4400 5650 50  0001 C CNN
 F 4 "0" H 4400 5650 50  0001 C CNN "JLCPCB BOM"
@@
 F 0 "D5" V 3896 6980 50  0000 R CNN
 F 1 "LED_B_V1" V 3805 6980 50  0000 R CNN
-F 2 "custom-pcb:LED_D5.0mm-centered" V 3850 7050 50  0001 C CNN
+F 2 "LED_SMD:LED_0603_1608Metric_Pad1.05x0.95mm_HandSolder" V 3850 7050 50  0001 C CNN
 F 3 "~" V 3850 7050 50  0001 C CNN
 F 4 "0" H 3850 7050 50  0001 C CNN "JLCPCB BOM"
@@
 F 0 "D7" V 4496 6980 50  0000 R CNN
 F 1 "LED_B_V2" V 4405 6980 50  0000 R CNN
-F 2 "custom-pcb:LED_D5.0mm-centered" V 4450 7050 50  0001 C CNN
+F 2 "LED_SMD:LED_0603_1608Metric_Pad1.05x0.95mm_HandSolder" V 4450 7050 50  0001 C CNN
 F 3 "~" V 4450 7050 50  0001 C CNN
 F 4 "0" H 4450 7050 50  0001 C CNN "JLCPCB BOM"
@@
 F 0 "D8" V 5096 6980 50  0000 R CNN
 F 1 "LED_B_V3" V 5005 6980 50  0000 R CNN
-F 2 "custom-pcb:LED_D5.0mm-centered" V 5050 7050 50  0001 C CNN
+F 2 "LED_SMD:LED_0603_1608Metric_Pad1.05x0.95mm_HandSolder" V 5050 7050 50  0001 C CNN
 F 3 "~" V 5050 7050 50  0001 C CNN
 F 4 "0" H 5050 7050 50  0001 C CNN "JLCPCB BOM"
@@
 F 0 "D10" V 5696 6980 50  0000 R CNN
 F 1 "LED_B_2H" V 5605 6980 50  0000 R CNN
-F 2 "custom-pcb:LED_D5.0mm-centered" V 5650 7050 50  0001 C CNN
+F 2 "LED_SMD:LED_0603_1608Metric_Pad1.05x0.95mm_HandSolder" V 5650 7050 50  0001 C CNN
 F 3 "~" V 5650 7050 50  0001 C CNN
 F 4 "0" H 5650 7050 50  0001 C CNN "JLCPCB BOM"
@@
 F 0 "D12" V 6296 6980 50  0000 R CNN
 F 1 "LED_B_4H" V 6205 6980 50  0000 R CNN
-F 2 "custom-pcb:LED_D5.0mm-centered" V 6250 7050 50  0001 C CNN
+F 2 "LED_SMD:LED_0603_1608Metric_Pad1.05x0.95mm_HandSolder" V 6250 7050 50  0001 C CNN
 F 3 "~" V 6250 7050 50  0001 C CNN
 F 4 "0" H 6250 7050 50  0001 C CNN "JLCPCB BOM"
@@
 F 0 "D9" V 5046 5580 50  0000 R CNN
 F 1 "LED_B_8H" V 4955 5580 50  0000 R CNN
-F 2 "custom-pcb:LED_D5.0mm-centered" V 5000 5650 50  0001 C CNN
+F 2 "LED_SMD:LED_0603_1608Metric_Pad1.05x0.95mm_HandSolder" V 5000 5650 50  0001 C CNN
 F 3 "~" V 5000 5650 50  0001 C CNN
 F 4 "0" H 5000 5650 50  0001 C CNN "JLCPCB BOM"
@@
 Connection ~ 6250 5950
 $Comp
-L Device:C_Small C?
+L Device:C_Small C18
 U 1 1 60B576BD
 P 5950 5850
-F 0 "C?" H 5858 5804 50  0000 R CNN
+F 0 "C18" H 5858 5804 50  0000 R CNN
 F 1 "0u1" H 5858 5895 50  0000 R CNN
-F 2 "" H 5950 5850 50  0001 C CNN
+F 2 "Capacitor_SMD:C_0402_1005Metric" H 5950 5850 50  0001 C CNN
 F 3 "~" H 5950 5850 50  0001 C CNN
 	1    5950 5850
@@
 Connection ~ 5600 5950
 $Comp
-L Device:C_Small C?
+L Device:C_Small C16
 U 1 1 60B6DFD4
 P 5300 5850
-F 0 "C?" H 5208 5804 50  0000 R CNN
+F 0 "C16" H 5208 5804 50  0000 R CNN
 F 1 "0u1" H 5208 5895 50  0000 R CNN
-F 2 "" H 5300 5850 50  0001 C CNN
+F 2 "Capacitor_SMD:C_0402_1005Metric" H 5300 5850 50  0001 C CNN
 F 3 "~" H 5300 5850 50  0001 C CNN
 	1    5300 5850
@@
 $EndComp
 $Comp
-L Device:C_Small C?
+L Device:C_Small C14
 U 1 1 60B74B0A
 P 4700 5850
-F 0 "C?" H 4608 5804 50  0000 R CNN
+F 0 "C14" H 4608 5804 50  0000 R CNN
 F 1 "0u1" H 4608 5895 50  0000 R CNN
-F 2 "" H 4700 5850 50  0001 C CNN
+F 2 "Capacitor_SMD:C_0402_1005Metric" H 4700 5850 50  0001 C CNN
 F 3 "~" H 4700 5850 50  0001 C CNN
 	1    4700 5850
@@
 Connection ~ 5000 5950
 $Comp
-L Device:C_Small C?
+L Device:C_Small C20
 U 1 1 60B89A22
 P 6600 7250
-F 0 "C?" H 6508 7204 50  0000 R CNN
+F 0 "C20" H 6508 7204 50  0000 R CNN
 F 1 "0u1" H 6508 7295 50  0000 R CNN
-F 2 "" H 6600 7250 50  0001 C CNN
+F 2 "Capacitor_SMD:C_0402_1005Metric" H 6600 7250 50  0001 C CNN
 F 3 "~" H 6600 7250 50  0001 C CNN
 	1    6600 7250
@@
 Connection ~ 6250 7350
 $Comp
-L Device:C_Small C?
+L Device:C_Small C19
 U 1 1 60B8FC2D
 P 5950 7250
-F 0 "C?" H 5858 7204 50  0000 R CNN
+F 0 "C19" H 5858 7204 50  0000 R CNN
 F 1 "0u1" H 5858 7295 50  0000 R CNN
-F 2 "" H 5950 7250 50  0001 C CNN
+F 2 "Capacitor_SMD:C_0402_1005Metric" H 5950 7250 50  0001 C CNN
 F 3 "~" H 5950 7250 50  0001 C CNN
 	1    5950 7250
@@
 $EndComp
 $Comp
-L Device:C_Small C?
+L Device:C_Small C17
 U 1 1 60B9047D
 P 5350 7250
-F 0 "C?" H 5258 7204 50  0000 R CNN
+F 0 "C17" H 5258 7204 50  0000 R CNN
 F 1 "0u1" H 5258 7295 50  0000 R CNN
-F 2 "" H 5350 7250 50  0001 C CNN
+F 2 "Capacitor_SMD:C_0402_1005Metric" H 5350 7250 50  0001 C CNN
 F 3 "~" H 5350 7250 50  0001 C CNN
 	1    5350 7250
@@
 Connection ~ 5650 7350
 $Comp
-L Device:C_Small C?
+L Device:C_Small C15
 U 1 1 60BAFCD4
 P 4750 7250
-F 0 "C?" H 4658 7204 50  0000 R CNN
+F 0 "C15" H 4658 7204 50  0000 R CNN
 F 1 "0u1" H 4658 7295 50  0000 R CNN
-F 2 "" H 4750 7250 50  0001 C CNN
+F 2 "Capacitor_SMD:C_0402_1005Metric" H 4750 7250 50  0001 C CNN
 F 3 "~" H 4750 7250 50  0001 C CNN
 	1    4750 7250
@@
 Connection ~ 4450 7350
 $Comp
-L Device:C_Small C?
+L Device:C_Small C13
 U 1 1 60BC1260
 P 4150 7250
-F 0 "C?" H 4058 7204 50  0000 R CNN
+F 0 "C13" H 4058 7204 50  0000 R CNN
 F 1 "0u1" H 4058 7295 50  0000 R CNN
-F 2 "" H 4150 7250 50  0001 C CNN
+F 2 "Capacitor_SMD:C_0402_1005Metric" H 4150 7250 50  0001 C CNN
 F 3 "~" H 4150 7250 50  0001 C CNN
 	1    4150 7250
@@
 $EndComp
 $Comp
-L Device:C_Small C?
+L Device:C_Small C12
 U 1 1 60BC1AB5
 P 3400 7250
-F 0 "C?" H 3308 7204 50  0000 R CNN
+F 0 "C12" H 3308 7204 50  0000 R CNN
 F 1 "0u1" H 3308 7295 50  0000 R CNN
-F 2 "" H 3400 7250 50  0001 C CNN
+F 2 "Capacitor_SMD:C_0402_1005Metric" H 3400 7250 50  0001 C CNN
 F 3 "~" H 3400 7250 50  0001 C CNN
 	1    3400 7250
@@
 $EndComp
 $Comp
-L Device:C_Small C?
+L Device:C_Small C11
 U 1 1 60BC3C1F
 P 2750 7250
-F 0 "C?" H 2658 7204 50  0000 R CNN
+F 0 "C11" H 2658 7204 50  0000 R CNN
 F 1 "0u1" H 2658 7295 50  0000 R CNN
-F 2 "" H 2750 7250 50  0001 C CNN
+F 2 "Capacitor_SMD:C_0402_1005Metric" H 2750 7250 50  0001 C CNN
 F 3 "~" H 2750 7250 50  0001 C CNN
 	1    2750 7250
@@
 $EndComp
 $Comp
-L Device:C_Small C?
+L Device:C_Small C10
 U 1 1 60BC4492
 P 2050 7250
-F 0 "C?" H 1958 7204 50  0000 R CNN
+F 0 "C10" H 1958 7204 50  0000 R CNN
 F 1 "0u1" H 1958 7295 50  0000 R CNN
-F 2 "" H 2050 7250 50  0001 C CNN
+F 2 "Capacitor_SMD:C_0402_1005Metric" H 2050 7250 50  0001 C CNN
 F 3 "~" H 2050 7250 50  0001 C CNN
 	1    2050 7250
@@
 $EndComp
 $Comp
-L Device:C_Small C?
+L Device:C_Small C9
 U 1 1 60BC4BA1
 P 1300 7250
-F 0 "C?" H 1208 7204 50  0000 R CNN
+F 0 "C9" H 1208 7204 50  0000 R CNN
 F 1 "0u1" H 1208 7295 50  0000 R CNN
-F 2 "" H 1300 7250 50  0001 C CNN
+F 2 "Capacitor_SMD:C_0402_1005Metric" H 1300 7250 50  0001 C CNN
 F 3 "~" H 1300 7250 50  0001 C CNN
 	1    1300 7250
@@
 	1300 6950 950  6950
 $Comp
-L Device:C_Small C?
+L Device:C_Small C21
 U 1 1 60AF2DD2
 P 6650 5850
-F 0 "C?" H 6558 5804 50  0000 R CNN
+F 0 "C21" H 6558 5804 50  0000 R CNN
 F 1 "0u1" H 6558 5895 50  0000 R CNN
-F 2 "" H 6650 5850 50  0001 C CNN
+F 2 "Capacitor_SMD:C_0402_1005Metric" H 6650 5850 50  0001 C CNN
 F 3 "~" H 6650 5850 50  0001 C CNN
 	1    6650 5850
@@
 Notes:\n22uF caps are only available in 0603 footprints at JLC\n100nF caps are available in 0402
 $Comp
-L Device:R_Small R?
+L Device:R_Small R28
 U 1 1 60D00276
 P 4500 2600
-F 0 "R?" V 4304 2600 50  0000 C CNN
+F 0 "R28" V 4304 2600 50  0000 C CNN
 F 1 "510R" V 4395 2600 50  0000 C CNN
-F 2 "" H 4500 2600 50  0001 C CNN
+F 2 "Resistor_SMD:R_0402_1005Metric" H 4500 2600 50  0001 C CNN
 F 3 "~" H 4500 2600 50  0001 C CNN
 	1    4500 2600
@@
 	4250 2600 4400 2600
 $Comp
-L Device:R_Small R?
+L Device:R_Small R29
 U 1 1 60D0BFA1
 P 4500 3250
-F 0 "R?" V 4304 3250 50  0000 C CNN
+F 0 "R29" V 4304 3250 50  0000 C CNN
 F 1 "510R" V 4395 3250 50  0000 C CNN
-F 2 "" H 4500 3250 50  0001 C CNN
+F 2 "Resistor_SMD:R_0402_1005Metric" H 4500 3250 50  0001 C CNN
 F 3 "~" H 4500 3250 50  0001 C CNN
 	1    4500 3250
@@
 	4250 3250 4400 3250
 $Comp
-L Device:R_Small R?
+L Device:R_Small R30
 U 1 1 60D3AD4D
 P 5650 2600
-F 0 "R?" V 5454 2600 50  0000 C CNN
+F 0 "R30" V 5454 2600 50  0000 C CNN
 F 1 "510R" V 5545 2600 50  0000 C CNN
-F 2 "" H 5650 2600 50  0001 C CNN
+F 2 "Resistor_SMD:R_0402_1005Metric" H 5650 2600 50  0001 C CNN
 F 3 "~" H 5650 2600 50  0001 C CNN
 	1    5650 2600
@@
 $EndComp
 $Comp
-L Device:R_Small R?
+L Device:R_Small R31
 U 1 1 60D3AE17
 P 5650 3250
-F 0 "R?" V 5454 3250 50  0000 C CNN
+F 0 "R31" V 5454 3250 50  0000 C CNN
 F 1 "510R" V 5545 3250 50  0000 C CNN
-F 2 "" H 5650 3250 50  0001 C CNN
+F 2 "Resistor_SMD:R_0402_1005Metric" H 5650 3250 50  0001 C CNN
 F 3 "~" H 5650 3250 50  0001 C CNN
 	1    5650 3250
@@
 $EndComp
 $Comp
-L Device:R_Small R?
+L Device:R_Small R32
 U 1 1 60D41ABE
 P 5650 3900
-F 0 "R?" V 5454 3900 50  0000 C CNN
+F 0 "R32" V 5454 3900 50  0000 C CNN
 F 1 "510R" V 5545 3900 50  0000 C CNN
-F 2 "" H 5650 3900 50  0001 C CNN
+F 2 "Resistor_SMD:R_0402_1005Metric" H 5650 3900 50  0001 C CNN
 F 3 "~" H 5650 3900 50  0001 C CNN
 	1    5650 3900
@@
 	5400 3900 5550 3900
 $Comp
-L Device:R_Small R?
+L Device:R_Small R33
 U 1 1 60D71D48
 P 6950 2600
-F 0 "R?" V 6754 2600 50  0000 C CNN
+F 0 "R33" V 6754 2600 50  0000 C CNN
 F 1 "510R" V 6845 2600 50  0000 C CNN
-F 2 "" H 6950 2600 50  0001 C CNN
+F 2 "Resistor_SMD:R_0402_1005Metric" H 6950 2600 50  0001 C CNN
 F 3 "~" H 6950 2600 50  0001 C CNN
 	1    6950 2600
@@
 $EndComp
 $Comp
-L Device:R_Small R?
+L Device:R_Small R34
 U 1 1 60D71E96
 P 6950 3250
-F 0 "R?" V 6754 3250 50  0000 C CNN
+F 0 "R34" V 6754 3250 50  0000 C CNN
 F 1 "510R" V 6845 3250 50  0000 C CNN
-F 2 "" H 6950 3250 50  0001 C CNN
+F 2 "Resistor_SMD:R_0402_1005Metric" H 6950 3250 50  0001 C CNN
 F 3 "~" H 6950 3250 50  0001 C CNN
 	1    6950 3250
